File: PCB/PiicoDev-Expansion-Board-for-Raspberry-Pi-Pico.kicad_sch (KiCad schematic)
At the start: 22 parts, among them J1 PiicoDev, J2 JST PH, J3 , J4 , Q1 MOSFET P-CH

Commit message: Wide voltage expansion board
Parts:
- removed FID1, FID2: Fiducial, Fiducial:Fiducial_1mm_Mask2mm, symbol Mechanical:Fiducial
- removed G1: LOGO_CoreElectronics_made-with-love, CoreElectronics_Artwork:CoreElectronics_logo_5mm, symbol CoreElectronics_Artwork:LOGO_CoreElectronics_made-with-love
- removed G2: LOGO_PiicoDev, CoreElectronics_Artwork:piicodev_logo_14.2x3.4mm, symbol CoreElectronics_Artwork:LOGO_PiicoDev
- added C1: 10uF, Capacitor_SMD:C_0805_2012Metric, symbol Device:C
- added C2, C3: 0.1uF, Capacitor_SMD:C_0603_1608Metric, symbol Device:C
- added C4, C5: 22uF, Capacitor_SMD:C_0603_1608Metric, symbol Device:C
- added L1: 10uF, Inductor_SMD:L_Abracon_ASPI-0630LR, symbol Device:L
- added R1: 100k, Resistor_SMD:R_0603_1608Metric, symbol Device:R
- added R2: 13.3k, Resistor_SMD:R_0603_1608Metric, symbol Device:R
- added U1: TPS54302, Package_TO_SOT_SMD:SOT-23-6, symbol Regulator_Switching:TPS54302
- H1, H2, H3, H4: footprint MountingHole:MountingHole_2.7mm_M2.5 -> MountingHole:MountingHole_3.2mm_M3
- J1: LCSC (none) -> C2845363
- J2: JLCPCB Rotation Offset (none) -> 180; LCSC (none) -> C47647
- J3, J4: JLCPCB Rotation Offset (none) -> 90; LCSC (none) -> C3975165
- Q1: LCSC (none) -> C15127
- R5, R6: footprint Resistor_SMD:R_0402_1005Metric -> Resistor_SMD:R_0603_1608Metric; LCSC (none) -> C23162
- R7, R8: footprint Resistor_SMD:R_0402_1005Metric -> Resistor_SMD:R_0603_1608Metric; LCSC (none) -> C22787
Connections:
- net GND: now also C1.2, C2.2, C4.2, C5.2, R2.2, U1.1 (GND)
- net I2C0_SCL: now also #U2.7 (GP5), J3.13 (Pin_13), J3.14 (Pin_14); no longer #U2.12 (GP9), J3.23 (Pin_23), J3.24 (Pin_24)
- net I2C0_SDA: now also #U2.6 (GP4), J3.11 (Pin_11), J3.12 (Pin_12); no longer #U2.11 (GP8), J3.21 (Pin_21), J3.22 (Pin_22)
- net VBAT: now also C1.1, C2.1, U1.3 (VIN); no longer Q1.3 (D)
- new net: #U2.11 (GP8), J3.21 (Pin_21), J3.22 (Pin_22)
- new net: #U2.12 (GP9), J3.23 (Pin_23), J3.24 (Pin_24)
- new net: C3.1, L1.1, U1.2 (SW)
- new net: R1.2, R2.1, U1.4 (FB)
- new net: C3.2, U1.6 (BOOT)
- new net +5V: C4.1, C5.1, L1.2, Q1.3 (D), R1.1
- no-connect marks 3 -> 4
Other:
- moved on the sheet: J2, Q1, R4

Commit message: prototype production
Parts:
- H1, H2, H3, H4, JP1, JP2, JP3: now left out of the parts list
- J1: LCSC C2845363 -> C160404
Changed lines of the file:
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@@
 			)
 		)
-		(property "LCSC" "C2845363"
+		(property "LCSC" "C160404"
 			(at 49.53 153.67 0)
 			(effects
@@
 		(unit 1)
 		(exclude_from_sim no)
-		(in_bom yes)
+		(in_bom no)
 		(on_board yes)
 		(dnp no)
@@
 		(unit 1)
 		(exclude_from_sim no)
-		(in_bom yes)
+		(in_bom no)
 		(on_board yes)
 		(dnp no)
@@
 		(unit 1)
 		(exclude_from_sim no)
-		(in_bom yes)
+		(in_bom no)
 		(on_board yes)
 		(dnp no)
@@
 		(unit 1)
 		(exclude_from_sim no)
-		(in_bom yes)
+		(in_bom no)
 		(on_board yes)
 		(dnp no)
@@
 		(unit 1)
 		(exclude_from_sim no)
-		(in_bom yes)
+		(in_bom no)
 		(on_board yes)
 		(dnp no)
@@
 		(unit 1)
 		(exclude_from_sim no)
-		(in_bom yes)
+		(in_bom no)
 		(on_board yes)
 		(dnp no)
@@
 		(unit 1)
 		(exclude_from_sim no)
-		(in_bom yes)
-		(on_board yes)
-		(dnp no)
+		(in_bom no)
+		(on_board yes)
+		(dnp no)
